File: v2_1/Seizo_Noise_v2.kicad_pcb (KiCad board)
At the start: 2 copper layers, 85 x 60 mm, 18 parts, among them J1 5V_IN (OSTTC022162), J3 PAM8302 INPUT, J4 SJ1-3533NG

Commit message: Candidate: route nine GND pads explicitly on B.Cu and validate natively
Routing:
- net GND: track 0.00 -> 216.7 mm
- added copper zone on B.Cu, net GND
